File: heatbed.brd (EAGLE design)
At the start: 188.9 x 423.3 mm, 0 parts

Commit message: modifying board to fit the pcb mill
Other:
- board size 188.9 x 423.3 mm -> 188.9 x 299.3 mm

Commit message: modifying for full 12 inch pcb
Other:
- board size 188.9 x 299.3 mm -> 188.9 x 305 mm

Commit message: swithing to 2.89mm trace width and the proper length to get 1.9 ohms resistance
Routing:
- net N$1: track 9203.8 -> 11368.5 mm
